File: MOTO_PCB/DebugProbe.kicad_sch (KiCad schematic)
At the start: 0 parts

Commit message: More routing
Parts:
- added C24, C25: 15p, Capacitor_SMD:C_0402_1005Metric, symbol Device:C
- added C26: 10u, Capacitor_SMD:C_0805_2012Metric, symbol Device:C
- added C27, C32: 10u, Capacitor_SMD:C_0603_1608Metric, symbol Device:C
- added C28, C29, C30, C33, C35, C36, C37, C38, C39, C40, C41, C42: 100n, Capacitor_SMD:C_0402_1005Metric, symbol Device:C
- added C31, C34: 1u, Capacitor_SMD:C_0402_1005Metric, symbol Device:C
- added CR2: BAT60JFILM, BAT60JFILM:CR_60JFILM_STM, symbol BAT60JFILM:BAT60JFILM
- added D1: RED, Diode_SMD:D_0402_1005Metric, symbol Device:LED
- added D2, D4: GREEN, Diode_SMD:D_0402_1005Metric, symbol Device:LED
- added D3, D5: YELLOW, Diode_SMD:D_0402_1005Metric, symbol Device:LED
- added J3: DebugnBoot, Connector_PinHeader_2.54mm:PinHeader_1x04_P2.54mm_Vertical, symbol Connector:Conn_01x04_Pin
- added J5: USB_C_Receptacle_USB2.0_14P, Connector_USB:USB_C_Receptacle_G-Switch_GT-USB-7010ASV, symbol Connector:USB_C_Receptacle_USB2.0_14P
- added J7: UART-PINS, Connector_PinHeader_2.54mm:PinHeader_1x03_P2.54mm_Vertical, symbol Connector:Conn_01x03_Pin
- added R17, R20: 1k, Resistor_SMD:R_0402_1005Metric, symbol Device:R
- added R18, R19: 5.1k, Resistor_SMD:R_0402_1005Metric, symbol Device:R_US
- added R21, R22: 27, Resistor_SMD:R_0402_1005Metric, symbol Device:R
- added R23, R31, R33: 470, Resistor_SMD:R_0402_1005Metric, symbol Device:R_US
- added R24, R25, R26, R27, R28, R29: 100, Resistor_SMD:R_0402_1005Metric, symbol Device:R_US
- added R30, R32: 2k, Resistor_SMD:R_0402_1005Metric, symbol Device:R_US
- added U10: USBLC6-2P6, Package_TO_SOT_SMD:SOT-666, symbol Power_Protection:USBLC6-2P6
- added U4: W25Q16JVUXIQ TR, W25Q16JVUXIQ:USON-8_UX_2x3x0p6_WIN, symbol W25Q16JVUXIQ:W25Q16JVUXIQ_TR
- added U5: AP2112K-3.3, Package_TO_SOT_SMD:SOT-23-5, symbol Regulator_Linear:AP2112K-3.3
- added U6: RP2040, Package_DFN_QFN:QFN-56-1EP_7x7mm_P0.4mm_EP3.2x3.2mm, symbol MCU_RaspberryPi_RP2040:RP2040
- added U7, U8: SN74AUP1T17DCKR, SN74AUP1T17DCKR:DCK5, symbol SN74AUP1T17DCKR:SN74AUP1T17DCKR
- added Y2: ABM8-272-T3, Crystal:Crystal_SMD_3225-4Pin_3.2x2.5mm, symbol Device:Crystal_GND24
Connections:
- new net: R22.2, U6.46 (USB_DM)
- new net: R21.2, U6.47 (USB_DP)
- new net: J7.1 (Pin_1), R24.2
- new net: J7.3 (Pin_3), R25.2, R26.2
- new net: D2.2 (A), R30.2
- new net: D1.2 (A), R23.2
- new net: C25.1, R20.2, Y2.3
- new net: D3.2 (A), R31.2
- new net: R29.1, U8.2 (A)
- new net: J5.A5 (CC1), R18.1
- new net: R26.1, U7.2 (A)
- new net: D4.2 (A), R32.2
- new net: J5.B5 (CC2), R19.1
- new net: J5.A7 (D-), J5.B7 (D-), U10.1 (I/O1)
- new net: J5.A6 (D+), J5.B6 (D+), U10.3 (I/O2)
- new net: D5.2 (A), R33.2
- new net: CR2.2, J5.A4 (VBUS), J5.A9 (VBUS), J5.B4 (VBUS), J5.B9 (VBUS)
- new net +P1V1: C28.1, C30.1, C31.1, U6.23 (DVDD), U6.45 (VREG_VOUT), U6.50 (DVDD)
- new net +P3V3: C27.1, C29.1, C32.1, C33.1, C34.1, C35.1, C36.1, C37.1, C38.1, C39.1, C40.1, C41.1, C42.1, U4.8 (VCC), U5.5 (VOUT), U6.1 (IOVDD), U6.10 (IOVDD), U6.22 (IOVDD), U6.33 (IOVDD), U6.42 (IOVDD), U6.43 (ADC_AVDD), U6.44 (VREG_IN), U6.48 (USB_VDD), U6.49 (IOVDD), U7.5 (VCC), U8.5 (VCC)
- new net GPIO0: U6.2 (GPIO0)
- new net GPIO1: U6.3 (GPIO1)
- new net GPIO10: U6.13 (GPIO10)
- new net GPIO11: U6.14 (GPIO11)
- new net GPIO12: R27.1, U6.15 (GPIO12)
- new net GPIO13: U6.16 (GPIO13), U8.4 (Y)
- new net GPIO14: R28.1, U6.17 (GPIO14)
- new net GPIO15: R32.1, U6.18 (GPIO15)
- new net GPIO16: R33.1, U6.27 (GPIO16)
- new net GPIO17: U6.28 (GPIO17)
- new net GPIO18: U6.29 (GPIO18)
- new net GPIO19: U6.30 (GPIO19)
- new net GPIO2: R23.1, U6.4 (GPIO2)
- new net GPIO20: U6.31 (GPIO20)
- new net GPIO21: U6.32 (GPIO21)
- new net GPIO22: U6.34 (GPIO22)
- new net GPIO23: U6.35 (GPIO23)
- new net GPIO24: U6.36 (GPIO24)
- new net GPIO25: U6.37 (GPIO25)
- new net GPIO26_ADC0: U6.38 (GPIO26_ADC0)
- new net GPIO27_ADC1: U6.39 (GPIO27_ADC1)
- new net GPIO28_ADC2: U6.40 (GPIO28_ADC2)
- new net GPIO29_ADC3: U6.41 (GPIO29_ADC3)
- new net GPIO3: U6.5 (GPIO3)
- new net GPIO4: R24.1, U6.6 (GPIO4)
- new net GPIO5: U6.7 (GPIO5), U7.4 (Y)
- new net GPIO6: R25.1, U6.8 (GPIO6)
- new net GPIO7: R30.1, U6.9 (GPIO7)
- new net GPIO8: R31.1, U6.11 (GPIO8)
- new net GPIO9: U6.12 (GPIO9)
- new net PGND: C24.2, C25.2, C26.2, C27.2, C28.2, C29.2, C30.2, C31.2, C32.2, C33.2, C34.2, C35.2, C36.2, C37.2, C38.2, C39.2, C40.2, C41.2, C42.2, D1.1 (K), D2.1 (K), D3.1 (K), D4.1 (K), D5.1 (K), J3.3 (Pin_3), J5.A1 (GND), J5.A12 (GND), J5.B1 (GND), J5.B12 (GND), J5.S1 (SHIELD), J7.2 (Pin_2), R18.2, R19.2, U10.2 (GND), U4.4 (GND), U5.2 (GND), U6.19 (TESTEN), U6.57 (GND), U7.3 (GND), U8.3 (GND), Y2.2, Y2.4
- new net PSWCLK: J3.2 (Pin_2), R27.2
- new net PSWD: J3.4 (Pin_4), R28.2, R29.2
- new net P_VBUS: C26.1, CR2.1, U10.5 (VBUS), U5.1 (VIN), U5.3 (EN)
- new net QSPI_SCLK: U4.6 (CLK), U6.52 (QSPI_SCLK)
- new net QSPI_SD0: U4.5 (DI(IO0)), U6.53 (QSPI_SD0)
- new net QSPI_SD1: U4.2 (DO(IO1)), U6.55 (QSPI_SD1)
- new net QSPI_SD2: U4.3 (/WP(IO2)), U6.54 (QSPI_SD2)
- new net QSPI_SD3: U4.7 (/HOLDOR/RESET(IO3)), U6.51 (QSPI_SD3)
- new net QSPI_SS: R17.1, U4.1 (/CS), U6.56 (QSPI_SS)
- new net USB_D+: R21.1, U10.4 (I/O2)
- new net USB_D-: R22.1, U10.6 (I/O1)
- new net XIN: C24.1, U6.20 (XIN), Y2.1
- new net XOUT: R20.1, U6.21 (XOUT)
- new net ~{USB_BOOT}: J3.1 (Pin_1), R17.2
- no-connect marks 0 -> 5
Other:
- note added: "Crystal"
- note added: "Debug LEDs and pins + BOOTSEL"
- note added: "ESD Protection"
- note added: "Flash"
- note added: "Make sure C10 is close to pin 44 of RP2040"
- note added: "Make sure C8 is close to pin 45 of RP2040"
- note added: "Make sure R3 and R4 are close to RP2040"
- note added: "Power"
- note added: "Probe Ready LED"
- note added: "UART Pins and LEDs"
