File: MOTO_PCB/MOTO_PCB.kicad_pcb (KiCad board)
At the start: 4 copper layers, 81 x 44.8 mm, 66 parts, among them J1 USB_C_Receptacle_USB2.0_14P, J2 Conn_01x14_Pin, J3 Conn_01x14_Pin, J4 Conn_01x14_Pin, J5 Conn_01x14_Pin, J6 Conn_01x03_Pin, J7 Conn_01x09_Socket, J8 Conn_01x09_Socket, SW1 BOOTSEL, SW2 RESET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

Commit message: More Vias
Routing:
- net +3V3: track 15.2 -> 44.3 mm, vias 1 -> 10
- net +1V1: track 3.35 -> 11.1 mm, vias 1 -> 3
- net /GPIO45_ADC5: track 0.00 -> 4.96 mm, vias 0 -> 1
- net /GPIO42_ADC2: track 0.00 -> 4.50 mm, vias 0 -> 1
- net /GPIO44_ADC4: track 0.00 -> 4.50 mm, vias 0 -> 1
- net /GPIO40_ADC0: track 0.00 -> 4.46 mm, vias 0 -> 1
- net /GPIO46_ADC6: track 0.00 -> 4.46 mm, vias 0 -> 1
- net /GPIO0: track 0.00 -> 4.43 mm, vias 0 -> 1
- net /GPIO1: track 0.00 -> 4.31 mm, vias 0 -> 1
- net /GPIO39: track 0.00 -> 4.13 mm, vias 0 -> 1
- net /GPIO47_ADC7: track 0.00 -> 3.77 mm, vias 0 -> 1
- net /RUN: track 0.00 -> 3.70 mm, vias 0 -> 1
- net /GPIO41_ADC1: track 0.00 -> 3.70 mm, vias 0 -> 1
- net /GPIO35: track 0.00 -> 3.65 mm, vias 0 -> 1
- net /GPIO37: track 0.00 -> 3.64 mm, vias 0 -> 1
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
Commit message: More line!
Routing:
- net /GPIO16: track 3.63 -> 61.9 mm
- net /GPIO11: track 4.72 -> 57.8 mm
- net /GPIO12: track 3.97 -> 56.9 mm
- net /GPIO13: track 4.36 -> 56.1 mm
- net /GPIO0: track 4.43 -> 55.3 mm
- net /GPIO6: track 1.60 -> 50.8 mm
- net /GPIO7: track 2.75 -> 49.9 mm
- net /GPIO5: track 2.42 -> 48.5 mm
- net /GPIO14: track 3.15 -> 47.3 mm
- net /GPIO4: track 2.06 -> 46.0 mm
- net /GPIO3: track 2.82 -> 45.9 mm
- net /GPIO2: track 3.18 -> 45.7 mm
- net /GPIO1: track 4.31 -> 46.0 mm
- net /GPIO15: track 3.23 -> 42.2 mm
- net /GPIO36: track 3.31 -> 34.7 mm
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
Commit message: Added parsing
Parts:
- moved R4 39.4 mm to (98.2, 98.5), turned to -90 degrees
- moved R1 32.4 mm to (90.0, 88.5), turned to -90 degrees
- moved R2 31.3 mm to (87.7, 87.5), turned to 180 degrees
- moved R5 31.1 mm to (87.0, 92.5), turned to 180 degrees
- moved U9 23.8 mm to (87.3, 89.9), turned to -90 degrees
- moved R3 19.1 mm to (77.2, 109.2), turned to -90 degrees
- moved C8 15.7 mm to (67.0, 99.5), turned to 90 degrees
- moved CR1 2.40 mm to (93.4, 88.5)
Routing:
- net VBUS: track 0.00 -> 201.0 mm
- net /GPIO21: track 22.0 -> 92.9 mm, vias 1 -> 5
- net /GPIO9: track 5.87 -> 74.4 mm, vias 1 -> 0
- net /GPIO8: track 52.2 -> 119.3 mm
- net /GPIO26: track 20.7 -> 86.8 mm, vias 1 -> 2
- net +3V3: track 43.4 -> 107.3 mm, vias 10 -> 20
- net /GPIO20: track 0.00 -> 58.0 mm, vias 0 -> 1
- net /SWCLK: track 0.00 -> 52.3 mm, vias 0 -> 1
- net /GPIO10: track 54.7 -> 103.6 mm
- net +1V1: track 24.8 -> 72.8 mm, vias 3 -> 4
- net /SWD: track 32.9 -> 70.0 mm
- net /GPIO19: track 26.1 -> 61.6 mm
- net /GPIO18: track 27.8 -> 54.8 mm
- net /RUN: track 3.70 -> 29.3 mm, vias 1 -> 2
- net UVBUS: track 0.00 -> 19.7 mm
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- added copper zone on In1.Cu, net +3V3
- removed copper zone on In1.Cu, net GND
Other:
- board text added: "Elise Bauerschmidt Sebastian Arhtur"
- board text added: "MOTOGPS"
